File: CAD/Eagle/Smart-LCD_1V1.brd (EAGLE design)
At the start: 99 x 67.7 mm, 53 parts, among them Q121 MMBT2222AL, U101 MEGA8-P, U401 TS4871ID, X131 LDR, X141 Switches, X151 LEDs, X201 LCD_23WAY__UC1608, X231 LED_A, X232 LED_K, X301 I2C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

Commit message: HW_V1.1 - LCD backlight - 1 ohms added to the NPN's emitter
Parts:
- added R122: 1R, rcl:R0805
Connections:
- new net LED_PWM_E: Q121.2, R122.1
- net GND: now also R122.2; no longer Q121.2
Changed lines of the file:
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@@
 <attribute name="VALUE" x="43.815" y="16.51" size="0.6096" layer="28" rot="MR90"/>
+</element>
+<element name="R122" library="rcl" package="R0805" value="1R" x="71.755" y="6.35" smashed="yes" rot="MR0">
+<attribute name="NAME" x="73.025" y="7.62" size="0.6096" layer="26" rot="MR0"/>
+<attribute name="VALUE" x="70.485" y="4.445" size="0.6096" layer="28" rot="MR0"/>
 </element>
 </elements>
@@
 <contactref element="R211" pad="1"/>
 <contactref element="C211" pad="2"/>
-<contactref element="Q121" pad="2"/>
 <wire x1="42.86" y1="1.765" x2="43" y2="1.905" width="0.254" layer="16"/>
 <wire x1="40.64" y1="8.57" x2="40.96" y2="8.89" width="0.3048" layer="16"/>
@@
 <via x="60.325" y="52.705" extent="1-16" drill="0.3"/>
 <via x="26.67" y="2.54" extent="1-16" drill="0.3"/>
-<via x="70.485" y="4.445" extent="1-16" drill="0.3"/>
-<via x="64.135" y="5.715" extent="1-16" drill="0.3"/>
+<via x="68.58" y="6.35" extent="1-16" drill="0.3"/>
+<via x="66.675" y="2.54" extent="1-16" drill="0.3"/>
 <via x="37.465" y="17.78" extent="1-16" drill="0.3"/>
 <via x="50.165" y="17.78" extent="1-16" drill="0.3"/>
@@
 <contactref element="R132" pad="1"/>
 <contactref element="D131" pad="3"/>
+<contactref element="R122" pad="2"/>
+<wire x1="94.615" y1="52.07" x2="92.5" y2="62.5" width="0" layer="19" extent="1-1"/>
+<wire x1="86.995" y1="52.07" x2="94.615" y2="52.07" width="0" layer="19" extent="1-1"/>
+<wire x1="80.01" y1="45.085" x2="86.995" y2="52.07" width="0" layer="19" extent="1-1"/>
+<wire x1="80.01" y1="37.465" x2="80.01" y2="45.085" width="0" layer="19" extent="1-1"/>
+<wire x1="82.61" y1="33.655" x2="80.01" y2="37.465" width="0" layer="19" extent="16-16"/>
+<wire x1="87.3" y1="31.75" x2="82.61" y2="33.655" width="0" layer="19" extent="16-16"/>
+<wire x1="90.805" y1="31.75" x2="87.3" y2="31.75" width="0" layer="19" extent="1-1"/>
+<wire x1="90.805" y1="33.34" x2="90.805" y2="31.75" width="0" layer="19" extent="16-16"/>
+<wire x1="77.41" y1="32.385" x2="82.61" y2="33.655" width="0" layer="19" extent="16-16"/>
+<wire x1="77.79" y1="29.845" x2="77.41" y2="32.385" width="0" layer="19" extent="16-16"/>
+<wire x1="75.565" y1="29.845" x2="77.79" y2="29.845" width="0" layer="19" extent="16-16"/>
+<wire x1="73.66" y1="32.07" x2="75.565" y2="29.845" width="0" layer="19" extent="16-16"/>
+<wire x1="68.58" y1="33.02" x2="73.66" y2="32.07" width="0" layer="19" extent="16-16"/>
+<wire x1="68.58" y1="30.795" x2="68.58" y2="33.02" width="0" layer="19" extent="16-16"/>
+<wire x1="64.77" y1="37.465" x2="68.58" y2="33.02" width="0" layer="19" extent="1-1"/>
+<wire x1="95.25" y1="27.305" x2="90.805" y2="31.75" width="0" layer="19" extent="1-1"/>
+<wire x1="70.485" y1="20.955" x2="68.58" y2="30.795" width="0" layer="19" extent="16-16"/>
+<wire x1="57.42" y1="30.48" x2="64.77" y2="37.465" width="0" layer="19" extent="1-1"/>
+<wire x1="53.34" y1="28.895" x2="57.42" y2="30.48" width="0" layer="19" extent="16-16"/>
+<wire x1="50.8" y1="28.895" x2="53.34" y2="28.895" width="0" layer="19" extent="16-16"/>
+<wire x1="53.02" y1="26.035" x2="53.34" y2="28.895" width="0" layer="19" extent="16-16"/>
+<wire x1="54.61" y1="20.955" x2="53.02" y2="26.035" width="0" layer="19" extent="16-16"/>
+<wire x1="59.055" y1="20.955" x2="54.61" y2="20.955" width="0" layer="19" extent="1-1"/>
+<wire x1="48.26" y1="33.655" x2="50.8" y2="28.895" width="0" layer="19" extent="16-16"/>
+<wire x1="50.165" y1="17.78" x2="54.61" y2="20.955" width="0" layer="19" extent="1-1"/>
+<wire x1="48.09" y1="18.415" x2="50.165" y2="17.78" width="0" layer="19" extent="16-16"/>
+<wire x1="44.135" y1="21.59" x2="48.09" y2="18.415" width="0" layer="19" extent="16-16"/>
+<wire x1="43.18" y1="26.035" x2="44.135" y2="21.59" width="0" layer="19" extent="16-16"/>
+<wire x1="37.465" y1="17.78" x2="44.135" y2="21.59" width="0" layer="19" extent="16-16"/>
+<wire x1="37.465" y1="11.11" x2="37.465" y2="17.78" width="0" layer="19" extent="16-16"/>
+<wire x1="40.64" y1="8.57" x2="37.465" y2="11.11" width="0" layer="19" extent="16-16"/>
+<wire x1="40.64" y1="6.665" x2="40.64" y2="8.57" width="0" layer="19" extent="16-16"/>
+<wire x1="43" y1="1.905" x2="40.64" y2="6.665" width="0" layer="19" extent="16-16"/>
+<wire x1="50.8" y1="41.275" x2="48.26" y2="33.655" width="0" layer="19" extent="1-1"/>
+<wire x1="50.8" y1="44.135" x2="50.8" y2="41.275" width="0" layer="19" extent="16-16"/>
+<wire x1="48.895" y1="52.705" x2="50.8" y2="44.135" width="0" layer="19" extent="16-16"/>
+<wire x1="43.815" y1="61.595" x2="48.895" y2="52.705" width="0" layer="19" extent="1-1"/>
+<wire x1="38.1" y1="61.595" x2="43.815" y2="61.595" width="0" layer="19" extent="1-1"/>
+<wire x1="33.02" y1="64.135" x2="38.1" y2="61.595" width="0" layer="19" extent="1-1"/>
+<wire x1="29.845" y1="63.815" x2="33.02" y2="64.135" width="0" layer="19" extent="16-16"/>
+<wire x1="35.56" y1="54.295" x2="38.1" y2="61.595" width="0" layer="19" extent="16-16"/>
+<wire x1="53.34" y1="64.135" x2="43.815" y2="61.595" width="0" layer="19" extent="1-1"/>
+<wire x1="58.42" y1="10.16" x2="59.055" y2="20.955" width="0" layer="19" extent="1-1"/>
+<wire x1="66.675" y1="2.54" x2="58.42" y2="10.16" width="0" layer="19" extent="1-1"/>
+<wire x1="68.58" y1="6.35" x2="66.675" y2="2.54" width="0" layer="19" extent="1-1"/>
+<wire x1="37.465" y1="36.83" x2="48.26" y2="33.655" width="0" layer="19" extent="1-1"/>
+<wire x1="34.29" y1="38.735" x2="37.465" y2="36.83" width="0" layer="19" extent="1-1"/>
+<wire x1="60.325" y1="52.705" x2="48.895" y2="52.705" width="0" layer="19" extent="1-1"/>
+<wire x1="66.04" y1="66.04" x2="53.34" y2="64.135" width="0" layer="19" extent="1-1"/>
+<wire x1="26.67" y1="2.54" x2="37.465" y2="11.11" width="0" layer="19" extent="16-16"/>
+<wire x1="86.995" y1="10.795" x2="68.58" y2="6.35" width="0" layer="19" extent="1-1"/>
+<wire x1="92.5" y1="7.5" x2="86.995" y2="10.795" width="0" layer="19" extent="1-1"/>
+<wire x1="7.5" y1="7.5" x2="26.67" y2="2.54" width="0" layer="19" extent="1-1"/>
+<wire x1="7.5" y1="62.5" x2="29.845" y2="63.815" width="0" layer="19" extent="16-16"/>
+<wire x1="3.81" y1="31.75" x2="7.5" y2="7.5" width="0" layer="19" extent="1-1"/>
+<wire x1="70.805" y1="6.35" x2="7.5" y2="7.5" width="0" layer="19" extent="1-1"/>
 </signal>
 <signal name="+5V">
@@
 <wire x1="71.12" y1="33.34" x2="71.12" y2="30.795" width="0.3048" layer="16"/>
 </signal>
+<signal name="LED_PWM_E">
+<contactref element="R122" pad="1"/>
+<contactref element="Q121" pad="2"/>
+<wire x1="72.705" y1="6.35" x2="72.56" y2="4.125" width="0" layer="19" extent="1-16"/>
+</signal>
 </signals>

Commit message: HW_V1.1 - df4iah_connector.lbr combined for Smart-LCD and FindMeSAT (2)
Parts:
- R122: value 1R -> 3R3
Changed lines of the file:
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@@
 <layers>
 <layer number="1" name="Top" color="4" fill="1" visible="yes" active="yes"/>
-<layer number="2" name="Route2" color="1" fill="3" visible="no" active="yes"/>
+<layer number="2" name="Route2" color="1" fill="3" visible="yes" active="yes"/>
 <layer number="3" name="Route3" color="4" fill="3" visible="no" active="no"/>
 <layer number="14" name="Route14" color="1" fill="6" visible="no" active="no"/>
-<layer number="15" name="Route15" color="4" fill="6" visible="no" active="yes"/>
+<layer number="15" name="Route15" color="4" fill="6" visible="yes" active="yes"/>
 <layer number="16" name="Bottom" color="1" fill="1" visible="yes" active="yes"/>
 <layer number="17" name="Pads" color="2" fill="1" visible="yes" active="yes"/>
@@
 <attribute name="VALUE" x="43.815" y="16.51" size="0.6096" layer="28" rot="MR90"/>
 </element>
-<element name="R122" library="rcl" package="R0805" value="1R" x="71.755" y="6.35" smashed="yes" rot="MR0">
+<element name="R122" library="rcl" package="R0805" value="3R3" x="71.755" y="6.35" smashed="yes" rot="MR0">
 <attribute name="NAME" x="73.025" y="7.62" size="0.6096" layer="26" rot="MR0"/>
 <attribute name="VALUE" x="70.485" y="4.445" size="0.6096" layer="28" rot="MR0"/>
