File: CAD/Eagle/Smart-LCD_1V0.brd (EAGLE design)
At the start: 99 x 67.7 mm, 49 parts, among them Q121 MMBT2222AL, U101 MEGA8-P, U221 MCP4018T-104E/LT, U401 TS4871ID, X131 LDR, X141 Switches, X151 LEDs, X201 LCD_23WAY__UC1608, X231 LED_A, X232 LED_K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

Commit message: CAD - minor corrections and PCB V1.0 ordering done
Connections:
- net +5V: now also X231.2
- net LED_K: now also X232.2
Changed lines of the file:
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@@
 <layer number="42" name="bRestrict" color="1" fill="10" visible="yes" active="yes"/>
 <layer number="43" name="vRestrict" color="2" fill="10" visible="yes" active="yes"/>
-<layer number="44" name="Drills" color="7" fill="1" visible="no" active="yes"/>
+<layer number="44" name="Drills" color="7" fill="1" visible="yes" active="yes"/>
 <layer number="45" name="Holes" color="7" fill="1" visible="yes" active="yes"/>
 <layer number="46" name="Milling" color="3" fill="1" visible="yes" active="yes"/>
@@
 <dimension x1="0" y1="0" x2="0" y2="67.7" x3="-8.5" y3="33.85" textsize="1.016" layer="47"/>
 <dimension x1="0" y1="67.7" x2="99" y2="67.7" x3="49.5" y3="76.015" textsize="1.016" layer="47"/>
-<text x="27.94" y="62.865" size="1.4224" layer="52" ratio="15" rot="MR0">Smart-LCD V1.0
+<text x="27.94" y="62.865" size="1.4224" layer="22" ratio="15" rot="MR0">Smart-LCD V1.0
 by DF4IAH</text>
-<text x="46.355" y="21.59" size="1.016" layer="26" ratio="12" rot="MR90">LDR</text>
+<text x="48.26" y="22.86" size="1.016" layer="26" ratio="12" rot="MR0">LDR</text>
 <text x="38.1" y="5.43" size="1.016" layer="21" ratio="12">LCD: MCCOG240128A6W-FPTLW</text>
 <text x="36.83" y="58.42" size="1.016" layer="26" ratio="12" rot="MR0">I2C</text>
-<text x="41.91" y="17.78" size="1.016" layer="26" ratio="12" rot="MR90">Switches</text>
+<text x="44.45" y="22.86" size="1.016" layer="26" ratio="12" rot="MR0">Switches</text>
 <text x="56.515" y="58.42" size="1.016" layer="26" ratio="12" rot="MR0">LEDs</text>
 <polygon width="0.1" layer="22">
@@
 <attribute name="PACKAGE" value="SOT-6" x="30.48" y="27.305" size="1.016" layer="28" rot="MR180" display="off"/>
 <attribute name="SUPPLIER" value="Microchip" x="30.48" y="27.305" size="1.016" layer="28" rot="MR180" display="off"/>
-<attribute name="NAME" x="34.6456" y="26.3652" size="0.6096" layer="26" ratio="10" rot="SMR0"/>
+<attribute name="NAME" x="34.925" y="26.67" size="0.6096" layer="26" ratio="10" rot="SMR0"/>
 <attribute name="VALUE" x="42.2148" y="23.749" size="0.6096" layer="28" ratio="10" rot="SMR0"/>
 </element>
@@
 </element>
 <element name="X131" library="df4iah_connector" package="1X02" value="LDR" x="46.99" y="26.035" smashed="yes" rot="MR0">
-<attribute name="NAME" x="48.895" y="25.4" size="1.016" layer="26" ratio="10" rot="MR90"/>
+<attribute name="NAME" x="48.26" y="30.48" size="1.016" layer="26" ratio="10" rot="MR0"/>
 <attribute name="VALUE" x="46.99" y="27.94" size="0.6096" layer="28" rot="MR270"/>
 </element>
@@
 <attribute name="VALUE" x="43.18" y="26.67" size="0.6096" layer="28" rot="MR0"/>
 </element>
-<element name="X232" library="df4iah_connector" package="P1-20X0.80" value="LED_K" x="79.35" y="2.505" locked="yes" smashed="yes">
+<element name="X232" library="df4iah_connector" package="P1-20X0.80" value="LED_K" x="79.35" y="2.505" smashed="yes">
 <attribute name="NAME" x="77.445" y="4.41" size="1.016" layer="25" ratio="10"/>
 <attribute name="VALUE" x="78.08" y="2.505" size="0.6096" layer="27"/>
 </element>
-<element name="X231" library="df4iah_connector" package="P1-20X0.80" value="LED_A" x="19.35" y="2.505" locked="yes" smashed="yes">
+<element name="X231" library="df4iah_connector" package="P1-20X0.80" value="LED_A" x="19.35" y="2.505" smashed="yes">
 <attribute name="NAME" x="17.445" y="4.41" size="1.016" layer="25" ratio="10"/>
 <attribute name="VALUE" x="18.08" y="2.505" size="0.6096" layer="27"/>
@@
 </element>
 <element name="X411" library="df4iah_connector" package="2X02" value="Audio" x="95.25" y="34.29" smashed="yes" rot="MR180">
-<attribute name="NAME" x="96.52" y="37.465" size="1.016" layer="26" ratio="10" rot="MR0"/>
+<attribute name="NAME" x="97.155" y="37.465" size="1.016" layer="26" ratio="10" rot="MR0"/>
 <attribute name="VALUE" x="92.71" y="34.925" size="1.016" layer="28" rot="MR180"/>
 </element>
@@
 <wire x1="35.56" y1="56.195" x2="35.56" y2="57.785" width="0.4064" layer="16"/>
 <wire x1="35.56" y1="57.785" x2="34.925" y2="58.42" width="0.4064" layer="16"/>
+<contactref element="X231" pad="2"/>
 </signal>
 <signal name="+3V3">
@@
 <wire x1="78.74" y1="2.54" x2="79.315" y2="2.54" width="0.8128" layer="16"/>
 <wire x1="79.315" y1="2.54" x2="79.35" y2="2.505" width="0.8128" layer="16"/>
+<contactref element="X232" pad="2"/>
 </signal>
 <signal name="LDR">

Commit message: CAD - changed value - C111 22nF --> 100 nF
Parts:
- C111: value 22nF -> 100nF
Changed lines of the file:
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@@
 <attribute name="VALUE" x="66.04" y="30.48" size="0.6096" layer="28" rot="MR270"/>
 </element>
-<element name="C111" library="rcl" package="C0805" value="22nF" x="68.58" y="29.845" smashed="yes" rot="MR90">
+<element name="C111" library="rcl" package="C0805" value="100nF" x="68.58" y="29.845" smashed="yes" rot="MR90">
 <attribute name="NAME" x="68.58" y="25.4" size="0.6096" layer="26" rot="MR90"/>
 <attribute name="VALUE" x="68.58" y="28.575" size="0.6096" layer="28" rot="MR90"/>

Commit message: CAD - I2C pull-ups changed to 1kR
Parts:
- R391, R392: value 1.5kR -> 1kR
Changed lines of the file:
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@@
 <attribute name="VALUE" x="36.195" y="62.23" size="0.6096" layer="28" rot="MR0"/>
 </element>
-<element name="R391" library="rcl" package="R0603" value="1.5kR" x="30.48" y="29.845" smashed="yes" rot="MR180">
+<element name="R391" library="rcl" package="R0603" value="1kR" x="30.48" y="29.845" smashed="yes" rot="MR180">
 <attribute name="NAME" x="31.75" y="31.115" size="0.6096" layer="26" rot="MR0"/>
 <attribute name="VALUE" x="31.75" y="29.21" size="0.6096" layer="28" rot="MR0"/>
 </element>
-<element name="R392" library="rcl" package="R0603" value="1.5kR" x="33.655" y="29.21" smashed="yes" rot="MR90">
+<element name="R392" library="rcl" package="R0603" value="1kR" x="33.655" y="29.21" smashed="yes" rot="MR90">
 <attribute name="NAME" x="34.925" y="27.94" size="0.6096" layer="26" rot="MR90"/>
 <attribute name="VALUE" x="33.02" y="27.94" size="0.6096" layer="28" rot="MR90"/>
