File: CAD/Eagle/Smart-LCD_1V0.sch (EAGLE design)
At the start: 27 parts, among them Q1 BC337-40, U101 MEGA32-P, U221 MCP4018T-104E/LT, X201 LCD_23WAY__UC1608, X301 I2C

Commit message: CAD - first layout worked on
Parts:
- removed Q1: BC337-40, df4iah_bipoltransistor:BC337-40
- added C131: 100pF, rcl:C-EUC0805
- added Q121: MMBT2222AL, df4iah_bipoltransistor:MMBT2222AL
- added R131: 33kR, rcl:R-EU_R0805
- added X131: LDR, df4iah_connector:HEADER-1X2
- R121: value 52kR -> 18kR
- R391, R392: value (none) -> 1.5kR
- renumbered TP1 to LED_A, TP2 to LED_K
Connections:
- net N$1 renamed AREF
- net N$2 renamed POT_A
- removed net LED_A: LED_A.TP, Q1.E
- removed net VDD: R222.2, U221.VDD, X201.8
- removed net VSS: C211.2, C221.2, LED_K.TP, R211.1, U221.VSS, X201.7
- new net LDR: C131.1, U101.(ADC0)PA0, X131.2
- new net LDR_P: R131.2, X131.1
- new net LED_K: LED_K.TP, Q121.C
- net !RST: now also U101.(SS)PB4
- net +3V3: now also R131.1, R222.2, U221.VDD, X201.8; no longer Q1.C
- net +5V: now also LED_A.TP
- net BM0: now also U101.(T1)PB1
- net BM1: now also U101.(T0/XCK)PB0
- net CD: now also U101.(MOSI)PB5
- net CS: now also U101.(AIN0/INT2)PB2
- net D0: now also U101.(RXD)PD0
- net D1: now also U101.(TXD)PD1
- net D2: now also U101.(INT0)PD2
- net D3: now also U101.(INT1)PD3
- net D4: now also U101.(OC1B)PD4
- net D5: now also U101.(OC1A)PD5
- net D6: now also U101.(ICP)PD6
- net D7: now also U101.(OC2)PD7
- net GND: now also C131.2, C211.2, C221.2, Q121.E, R211.1, U221.VSS, X201.7
- net LED_PWM_B: now also Q121.B; no longer Q1.B
- net VBIAS: now also R221.2
- net WR0: now also U101.(MISO)PB6
- net WR1: now also U101.(SCK)PB7
Other:
- note added: "LDR"
- moved on the sheet: C221

Commit message: CAD - routed, but audio amplifier still TODO
Parts:
- removed LED_A, LED_K: TPPAD1-20, df4iah_connector:TPPAD1-20
- added C141: 100pF, rcl:C-EUC0805
- added H411, H412: MOUNT-HOLE1.7, df4iah_holes:MOUNT-HOLE1.7
- added R141: 18kR, rcl:R-EU_R0805
- added R151, R152: 330R, rcl:R-EU_R0805
- added X141: Switches, df4iah_connector:HEADER-2X2
- added X151: LEDs, df4iah_connector:HEADER-2X2
- added X231: LED_A, df4iah_connector:CON_1X
- added X232: LED_K, df4iah_connector:CON_1X
- U101: value MEGA32-P -> MEGA8-P; device df4iah_processors:MEGA32-P -> df4iah_processors:MEGA8-P
Connections:
- removed net !RESET: R101.1, U101.RESET
- removed net BM0: U101.(T1)PB1, X201.22
- removed net BM1: U101.(T0/XCK)PB0, X201.23
- new net AG: R152.1, X151.3
- new net AG_D: R152.2, U101.PB7(XTAL2/TOSC2)
- new net AR: R151.1, X151.2
- new net AR_D: R151.2, U101.PB6(XTAL1/TOSC1)
- new net AUDIO_D: R141.1, U101.PB1(OC1A)
- new net AUDIO_LP: C141.1, R141.2
- new net SW_I: U101.PC1(ADC1), X141.2
- new net SW_P: U101.PB2(SS/OC1B), X141.3
- new net SW_Q: U101.PC2(ADC2), X141.4
- net !RST: now also R101.2, U101.PC6(/RESET); no longer U101.(SS)PB4
- net +3V3: now also R101.1, U101.VCC@1, X201.22, X201.23; no longer R101.2, U101.VCC
- net +5V: now also X231.1; no longer LED_A.TP
- net AREF: now also C111.2; no longer C111.1
- net CD: now also U101.PB0(ICP); no longer U101.(MOSI)PB5
- net CS: now also U101.PC3(ADC3); no longer U101.(AIN0/INT2)PB2
- net D0: now also U101.PD0(RXD); no longer U101.(RXD)PD0
- net D1: now also U101.PD1(TXD); no longer U101.(TXD)PD1
- net D2: now also U101.PD2(INT0); no longer U101.(INT0)PD2
- net D3: now also U101.PD3(INT1); no longer U101.(INT1)PD3
- net D4: now also U101.PD4(XCK/T0); no longer U101.(OC1B)PD4
- net D5: now also U101.PD5(T1); no longer U101.(OC1A)PD5
- net D6: now also U101.PD6(AIN0); no longer U101.(ICP)PD6
- net D7: now also U101.PD7(AIN1); no longer U101.(OC2)PD7
- net GND: now also C111.1, C141.2, U101.GND@1, X141.1, X151.1; no longer C111.2, U101.GND
- net LDR: now also U101.PC0(ADC0); no longer U101.(ADC0)PA0
- net LED_K: now also X232.1; no longer LED_K.TP
- net LED_PWM_D: now also U101.PB3(MOSI/OC2); no longer U101.(AIN1/OC0)PB3
- net SCL: now also U101.PC5(ADC5/SCL); no longer U101.(SCL)PC0
- net SDA: now also U101.PC4(ADC4/SDA); no longer U101.(SDA)PC1
- net WR0: now also U101.PB4(MISO); no longer U101.(MISO)PB6
- net WR1: now also U101.PB5(SCK); no longer U101.(SCK)PB7
Other:
- note added: "BM0"
- note added: "BM1"
- note added: "Contacts"
- note added: "LEDs"
- moved on the sheet: C102, C111, C131, Q121, R101, R121, R131, X131

Commit message: CAD - audio amplifier added, but CPU must be placed on the solder side
Parts:
- removed C141: 100pF, rcl:C-EUC0805
- removed H401, H402, H403, H404: MOUNT-PAD-ROUND2.8, holes:MOUNT-PAD-ROUND2.8
- removed H411, H412: MOUNT-HOLE1.7, df4iah_holes:MOUNT-HOLE1.7
- added C103: 100pF, rcl:C-EUC0805
- added C401: 22uF, rcl:C-EUC0805
- added C402: 100nF, rcl:C-EUC0805
- added C411, C412: 47uF, rcl:C-EUC0805
- added C431: 1uF, rcl:C-EUC0805
- added C452: 470pF, rcl:C-EUC0805
- added C455: 470nF, rcl:C-EUC0805
- added H501, H502, H503, H504: MOUNT-PAD-ROUND2.8, holes:MOUNT-PAD-ROUND2.8
- added H511, H512: MOUNT-HOLE1.7, df4iah_holes:MOUNT-HOLE1.7
- added R451, R454: 22kR, rcl:R-EU_R0805
- added U401: TS4871ID, df4iah_opamp:TS4871ID
- added X411: Audio, df4iah_connector:HEADER-2X2
- C111: value 100pF -> 22nF
- R111: value 18kR -> 3.3kR
- renumbered R141 to R111
Connections:
- new net AU454: C455.1, R454.2
- new net BYPASS: C431.1, U401A.BYPASS, U401A.VIN_P
- new net SPK_N: C412.2, X411.2
- new net SPK_P: C411.2, X411.1
- new net VIN_N: C452.1, C455.2, R451.1, U401A.VIN_N
- new net VOUT1: C411.1, C452.2, R451.2, U401A.VOUT1
- new net VOUT2: C412.1, U401A.VOUT2
- net +3V3: now also C401.1, C402.1, U401B.VCC
- net AREF: now also C103.2; no longer C111.2
- net AUDIO_LP: now also C111.1, R454.1; no longer C141.1
- net GND: now also C103.1, C111.2, C401.2, C402.2, C431.2, H501.MOUNT, H502.MOUNT, H503.MOUNT, H504.MOUNT, U401A.STANDBY, U401B.VSS; no longer C111.1, C141.2, H401.MOUNT, H402.MOUNT, H403.MOUNT, H404.MOUNT
Other:
- note added: "Audio"

Commit message: CAD - changed value - C111 22nF --> 100 nF
Parts:
- C111: value 22nF -> 100nF
Other:
- note added: "EN"
- note added: "RD/!WR"
- moved on the sheet: C101, C102, C103, C111, C131, H501, H502, H503, H504, H511, H512, Q121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

Commit message: CAD - I2C pull-ups changed to 1kR
Parts:
- R391, R392: value 1.5kR -> 1kR
Changed lines of the file:
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@@
 <part name="+3V3_301" library="df4iah_supply" deviceset="+3V3" device=""/>
 <part name="+5V0_301" library="df4iah_supply" deviceset="+5V" device=""/>
-<part name="R391" library="rcl" deviceset="R-EU_" device="R0603" value="1.5kR"/>
-<part name="R392" library="rcl" deviceset="R-EU_" device="R0603" value="1.5kR"/>
+<part name="R391" library="rcl" deviceset="R-EU_" device="R0603" value="1kR"/>
+<part name="R392" library="rcl" deviceset="R-EU_" device="R0603" value="1kR"/>
 <part name="FRAME4" library="df4iah_frame" deviceset="A4L-LOC" device="" value="Holes"/>
 <part name="X201" library="df4iah_connector" deviceset="LCD_23WAY__UC1608" device=""/>

Commit message: HW_V1.0 - do not place I2C poti
Other:
- note added: "do not place U221 and R222"
Changed lines of the file:
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@@
 <text x="157.48" y="121.92" size="1.778" layer="97" rot="R90">BM1</text>
 <text x="154.94" y="121.92" size="1.778" layer="97" rot="R90">BM0</text>
+<text x="154.94" y="68.58" size="1.778" layer="97">do not place U221 and R222</text>
 </plain>
 <instances>
